Commit message: connection with between sycl and ros success, and fpga version of stomp is success

File: install/my_bot/share/my_bot/description/robot.urdf.xacro (robot description, xacro)
@@ -120,5 +120,5 @@
         <child link="link_1"/>
         <axis xyz="0.0 0.0 1"/>
-        <limit lower="0.0" upper="${M_PI * 2}" effort="300.0" velocity="1.0"/>
+        <limit lower="${-M_PI }" upper="${M_PI * 2}" effort="300.0" velocity="1.0"/>
     </joint>
     <!--=============================================================================-->
@@ -173,5 +173,5 @@
         <child link="link_2"/>
         <axis xyz="1.0 0.0 0.0"/>
-        <limit lower="0.0" upper="${M_PI * 2}" effort="300.0" velocity="1.0"/>
+        <limit lower="${-M_PI }" upper="${M_PI * 2}" effort="300.0" velocity="1.0"/>
     </joint>
     <!--=============================================================================-->
@@ -225,5 +225,5 @@
         <child link="link_3"/>
         <axis xyz="1.0 0.0 0.0"/>
-        <limit lower="0.0" upper="${M_PI * 2}" effort="300.0" velocity="1.0"/>
+        <limit lower="${-M_PI }" upper="${M_PI * 2}" effort="300.0" velocity="1.0"/>
     </joint>
     <!--=============================================================================-->
@@ -251,5 +251,5 @@
         <child link="link_4"/>
         <axis xyz="0.0 0.0 01.0"/>
-        <limit lower="0.0" upper="${M_PI * 2}" effort="300.0" velocity="1.0"/>
+        <limit lower="${-M_PI}" upper="${M_PI * 2}" effort="300.0" velocity="1.0"/>
     </joint>
     <!--=============================================================================-->
@@ -355,6 +355,6 @@
     <xacro:transmission_block joint_name="gripper_joint_2"/> -->
     <!-- ros_control plugin -->
-    <xacro:property name="steer_limlow" value="-1.5"/>
-    <xacro:property name="steer_limhigh" value="1.5"/>
+    <xacro:property name="steer_limlow" value="-3.14"/>
+    <xacro:property name="steer_limhigh" value="3.14"/>
     <ros2_control name="GazeboSimSystem" type="system">
         <hardware>
@@ -363,6 +363,6 @@
         <joint name="joint_1">
             <command_interface name = "position">
-                <param name="min">-1.5</param>
-                <param name="max">1.5</param>
+               <param name="min">${steer_limlow}</param>
+               <param name="min">${steer_limhigh}</param>
             </command_interface>
             <state_interface name="position"/>
@@ -388,4 +388,13 @@
             <state_interface name="effort"/>
         </joint>
+            <!-- <joint name="gripper_joint_1">
+            <command_interface name = "position">
+                <param name="min">${steer_limlow}</param>
+                <param name="max">${steer_limhigh}</param>
+            </command_interface>
+            <state_interface name="position"/>
+            <state_interface name="velocity"/>
+            <state_interface name="effort"/>
+        </joint> -->
     </ros2_control>
         <gazebo>
